File: CHIP_POCKET_C.brd (EAGLE design)
At the start: 161.7 x 109.3 mm, 74 parts, among them IC1 74AHC1G08DCK, J1 98401-801-40LF, J3 S2B-PH-SM4-TB, Q3 MOSFET-PCHANNEL, Q4 MOSFET-PCHANNEL, U3 DS2431P, U4 MMA8452Q, U5 NCP5623DTBR2G, X1 FH12-40S-0.5SH

Commit message: added hub
Parts:
- removed FD2, FD3: FIDUCIAL, Keyboard v0.3:FIDUCIAL_1MM
- added C21: 10nF/50V, rcl:C0805
- added C22: 2.2nF, rcl:C0805
- added C23, C24, C30, C31: VJ1210V106ZXJTW1BC, rcl:C1210
- added C25: 10uF/25V, rcl:C1210
- added C26, C27, C28, C29: n.a., rcl:C1210
- added C32: 100nF, rcl:C0805
- added C33, C34: 22pF, rcl:C0805
- added D1, D3, D4: ES2D, diode:SMB
- added DATA_USB: USBUSB-MICROB-SMT-DIP, Spark:USB-MICROB-SMT-DIP
- added L1: SRN6045-100M, Keyboard v0_5:SRN6045
- added LED2, LED3, LED4, LED5, LED6: 150080BS75000, led:CHIP-LED0805
- added PAD1, PAD2: WIREPAD3,17/1,3, wirepad:3,17/1,3
- added Q1: FOXSDLF/120-20, adafruit:SM49
- added R10: 2.7k, rcl:R0805
- added R11, R13, R3: 10k, rcl:R0805
- added R14, R15, R19: ERJ-6ENF3300V, rcl:R0805
- added R2: 15k, rcl:R0805
- added R9: 28.7k, rcl:R0805
- added U$12: ACT4060ASHDEFAULT, JKW_CHIP:SOP-8
- added U$13: FE1.1S, imcom:FE1.1S_SSOP-28
- added VD1, VD2, VD3: n.a., usblc6:SOT-23-6L
- added X2, X3, X4, X5: USB-A-HU, con-usb:USB-A-HU
- J1: value 98401-801-40LF -> 2X20-CHIP2X20-SMT-CHIP; device PocketCHIP-v1.0:98401-801-40LF -> JKW_CHIP:2XAWHW40_G_SMD_R
- moved G 59.2 mm to (49.0, 9.91)
- moved J1 45.4 mm to (77.8, 69.6), flipped to the top, turned to 270 degrees
- moved RO 6.18 mm to (116.1, 20.3)
- moved RI 6.10 mm to (116.1, 22.6)
- moved C1 4.83 mm to (109.0, 21.1)
- moved C2 4.83 mm to (115.6, 13.7)
- moved C20 4.83 mm to (102.1, 15.5)
- moved C3 4.83 mm to (102.1, 13.5)
- moved PAM1 4.83 mm to (108.7, 14.2)
- moved JP1 4.13 mm to (149.1, 89.2)
- moved LO 3.09 mm to (124.0, 20.1)
- moved LI 3.05 mm to (124.0, 22.4)
- moved R12 3.05 mm to (111.4, 76.4)
- moved U3 2.90 mm to (110.4, 81.6)
- moved C5 2.84 mm to (121.7, 19.3)
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Connections:
- new net CHR: C23.2, C24.2, D4.A, J1.CHG-IN, L1.P$1
- new net DM1: U$13.10, VD1.3, X5.D-
- new net DM2: U$13.8, VD1.6, X4.D-
- new net DM3: U$13.6, VD2.3, X3.D-
- new net DM4: U$13.4, VD2.6, X2.D-
- new net DMU: DATA_USB.D-, U$13.15, VD3.4
- new net DP1: U$13.11, VD1.1, X5.D+
- new net DP2: U$13.9, VD1.4, X4.D+
- new net DP3: U$13.7, VD2.1, X3.D+
- new net DP4: U$13.5, VD2.4, X2.D+
- new net DPU: DATA_USB.D+, U$13.16, VD3.6
- new net N$64: D3.A, PAD1.1
- new net N$65: C21.2, D1.C, L1.P$2, U$12.3
- new net N$66: C21.1, U$12.1
- new net N$67: C22.2, R2.1
- new net N$68: C22.1, U$12.6
- new net N$69: R3.1, R9.2, U$12.5
- new net N$70: C31.2, U$13.13, U$13.21
- new net N$71: C30.2, U$13.12, U$13.28
- new net N$72: R10.2, U$13.14
- new net N$73: R13.2, U$13.17
- new net N$74: R11.2, U$13.19
- new net N$75: C33.1, Q1.2, U$13.2
- new net N$76: C34.1, Q1.1, U$13.3
- new net N$77: LED6.C, R19.1
- new net N$78: LED4.C, LED5.A, R15.1
- new net N$79: LED2.A, LED3.C, R14.1
- new net N$80: LED2.C, LED3.A, LED4.A, LED5.C, LED6.A, U$13.22
- new net N$81: R14.2, U$13.24
- new net N$82: R15.2, U$13.23
- new net VCC: C26.2, C27.2, C28.2, C29.2, C32.2, D4.C, R11.1, R13.1, R9.1, U$13.20, U$13.25, U$13.26, VD1.5, VD2.5, VD3.5, X2.VBUS, X3.VBUS, X4.VBUS, X5.VBUS
- new net VCC-1V8: J1.VCC1V8
- new net VIN: C25.2, D3.C, U$12.2
- new net V_UP: DATA_USB.VBUS, U$13.18
- net 1WIRE: now also J1.LCD-D2; no longer J1.58
- net ADC: now also J1.LRADC; no longer J1.12
- net AUDIO_L: now also J1.HPL; no longer J1.3
- net AUDIO_R: now also J1.HPR; no longer J1.7
- net DCLK: now also J1.LCD-CLK; no longer J1.76
- net EN: now also J1.LCD-D18; no longer J1.70
- net FEL: now also J1.FEL; no longer J1.8
- net GND: now also C23.1, C24.1, C25.1, C26.1, C27.1, C28.1, C29.1, C30.1, C31.1, C32.1, C33.2, C34.2, D1.A, DATA_USB.GND, DATA_USB.MT1, DATA_USB.MT2, J1.GND@1, J1.GND@10, J1.GND@2, J1.GND@3, J1.GND@4, J1.GND@5, J1.GND@6, J1.GND@7, J1.GND@8, PAD2.1, R10.1, R19.2, R3.2, U$12.4, U$13.1, VD1.2, VD2.2, VD3.2, X2.GND, X3.GND, X4.GND, X5.GND; no longer J1.2, J1.21, J1.22, J1.39, J1.40, J1.42, J1.43, J1.51, J1.80
- net GP1: now also J1.XIO-P2; no longer J1.16
- net GP2: now also J1.XIO-P3; no longer J1.15
- net GP3: now also J1.XIO-P4; no longer J1.18
- net GP4: now also J1.XIO-P5; no longer J1.17
- net GP5: now also J1.XIO-P6; no longer J1.20
- net GP6: now also J1.XIO-P7; no longer J1.19
- net HSYNC: now also J1.LCD-HSYNC; no longer J1.77
- net I2C-SCL: now also J1.TWI2-SCK; no longer J1.25
- net I2C-SDA: now also J1.TWI2-SDA; no longer J1.26
- net KPD_I2C_SCL: now also J1.TWI1-SCK; no longer J1.52
- net KPD_I2C_SDA: now also J1.TWI1-SDA; no longer J1.50
- net KPD_INT: now also J1.AP-EINT1; no longer J1.24
- net LCD_D10: now also J1.LCD-D10; no longer J1.64
- net LCD_D11: now also J1.LCD-D11; no longer J1.65
- net LCD_D12: now also J1.LCD-D12; no longer J1.66
- net LCD_D13: now also J1.LCD-D13; no longer J1.67
- net LCD_D14: now also J1.LCD-D14; no longer J1.68
- net LCD_D15: now also J1.LCD-D15; no longer J1.69
- net LCD_D19: now also J1.LCD-D19; no longer J1.71
- net LCD_D20: now also J1.LCD-D20; no longer J1.72
- net LCD_D21: now also J1.LCD-D21; no longer J1.73
- net LCD_D22: now also J1.LCD-D22; no longer J1.74
- net LCD_D23: now also J1.LCD-D23; no longer J1.75
- net LCD_D3: now also J1.LCD-D3; no longer J1.59
- net LCD_D4: now also J1.LCD-D4; no longer J1.60
- net LCD_D5: now also J1.LCD-D5; no longer J1.61
- net LCD_D6: now also J1.LCD-D6; no longer J1.62
- net LCD_D7: now also J1.LCD-D7; no longer J1.63
- net LCD_DE: now also J1.LCD-DE; no longer J1.79
- net LCD_XL: now also J1.X1; no longer J1.54
- net LCD_XR: now also J1.X2; no longer J1.53
- net LCD_YD: now also J1.Y2; no longer J1.55
- net LCD_YU: now also J1.Y1; no longer J1.56
- net PWM: now also J1.PWM0; no longer J1.57
- net PWR_ON: now also J1.PWRON; no longer J1.49
- net SDIO_CARD: now also J1.AP-EINT3; no longer J1.23
- net SDIO_CLK: now also J1.CSID5; no longer J1.35
- net SDIO_CMD: now also J1.CISD4; no longer J1.36
- net SDIO_DAT0: now also J1.CSID0; no longer J1.32
- net SDIO_DAT1: now also J1.CSID1; no longer J1.31
- net SDIO_DAT2: now also J1.CSID2; no longer J1.34
- net SDIO_DAT3: now also J1.CSID3; no longer J1.33
- net SPI-CLK: now also J1.CSICK; no longer J1.27
- net SPI-MISO: now also J1.CSIVSYNC; no longer J1.29
- net SPI-MOSI: now also J1.CSIHYSYNC; no longer J1.30
- net SPI-SEL: now also J1.CSPICK; no longer J1.28
- net UART_RX: now also J1.UART1-RX; no longer J1.6
- net UART_TX: now also J1.UART1-TX; no longer J1.4
- net VBAT_EXT: now also J1.BAT; no longer J1.47
- net VCC3V3: now also J1.VCC3V3@1, J1.VCC3V3@2; no longer J1.10, J1.46
- net VCC5V: now also J1.VCC-5V@1, J1.VCC-5V@2; no longer J1.1, J1.44
- net VSYNC: now also J1.LCD-VSYNC; no longer J1.78
Routing:
- net CHR: track 0.00 -> 160.7 mm
- net VCC: track 0.00 -> 104.5 mm, vias 0 -> 5
- net GND: track 90.7 -> 171.3 mm, vias 155 -> 151
- net DPU: track 0.00 -> 54.0 mm, vias 0 -> 2
- net DMU: track 0.00 -> 52.8 mm, vias 0 -> 2
- net DM4: track 0.00 -> 47.6 mm, vias 0 -> 3
- net N$82: track 0.00 -> 45.1 mm, vias 0 -> 2
- net DM2: track 0.00 -> 41.9 mm, vias 0 -> 2
- net DM3: track 0.00 -> 41.1 mm, vias 0 -> 2
- net DM1: track 0.00 -> 37.9 mm
- net DP1: track 0.00 -> 37.6 mm
- net N$81: track 0.00 -> 36.1 mm, vias 0 -> 2
- net DP2: track 0.00 -> 34.8 mm
- net N$69: track 0.00 -> 33.4 mm
- net N$80: track 0.00 -> 33.1 mm, vias 0 -> 2
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