File: CHIP_POCKET_C.sch (EAGLE design)
At the start: 74 parts, among them IC1 74AHC1G08DCK, J1 98401-801-40LF, J3 S2B-PH-SM4-TB, Q3 MOSFET-PCHANNEL, Q4 MOSFET-PCHANNEL, U3 DS2431P, U4 MMA8452Q, U5 NCP5623DTBR2G, X1 FH12-40S-0.5SH

Commit message: added hub
Parts:
- removed FD2, FD3: FIDUCIAL, Keyboard v0.3:FIDUCIAL
- added C21: 10nF/50V, rcl:C-EUC0805
- added C22: 2.2nF, rcl:C-EUC0805
- added C23, C24, C30, C31: VJ1210V106ZXJTW1BC, rcl:C-EUC1210
- added C25: 10uF/25V, rcl:C-EUC1210
- added C26, C27, C28, C29: n.a., rcl:C-EUC1210
- added C32: 100nF, rcl:C-EUC0805
- added C33, C34: 22pF, rcl:C-EUC0805
- added D1, D3, D4: ES2D, diode:ES2D
- added DATA_USB: USBUSB-MICROB-SMT-DIP, Spark:USBUSB-MICROB-SMT-DIP
- added L1: SRN6045-100M, Keyboard v0_5:SRN6045-100M
- added LED2, LED3, LED4, LED5, LED6: 150080BS75000, led:LEDCHIP-LED0805
- added PAD1, PAD2: WIREPAD3,17/1,3, wirepad:WIREPAD3,17/1,3
- added Q1: FOXSDLF/120-20, adafruit:CRYSTALSM49
- added R10: 2.7k, rcl:R-EU_R0805
- added R11, R13, R3: 10k, rcl:R-EU_R0805
- added R14, R15, R19: ERJ-6ENF3300V, rcl:R-EU_R0805
- added R2: 15k, rcl:R-EU_R0805
- added R9: 28.7k, rcl:R-EU_R0805
- added U$12: ACT4060ASHDEFAULT, JKW_CHIP:ACT4060ASHDEFAULT
- added U$13: FE1.1S, imcom:FE1.1S
- added VD1, VD2, VD3: n.a., usblc6:USBLC6-4SC6
- added X2, X3, X4, X5: USB-A-HU, con-usb:USB-A-HU
- J1: value 98401-801-40LF -> 2X20-CHIP2X20-SMT-CHIP; device PocketCHIP-v1.0:98401-801-40LF -> JKW_CHIP:2X20-CHIP2X20-SMT-CHIP
Connections:
- new net CHR: C23.2, C24.2, D4.A, J1.ACIN-5V, L1.1
- new net DM1: U$13.DM1, VD1.I/O2, X5.D+
- new net DM2: U$13.DM2, VD1.I/O4, X4.D+
- new net DM3: U$13.DM3, VD2.I/O2, X3.D+
- new net DM4: U$13.DM4, VD2.I/O4, X2.D+
- new net DMU: DATA_USB.D-, U$13.DMU, VD3.I/O3
- new net DP1: U$13.DP1, VD1.I/O1, X5.D-
- new net DP2: U$13.DP2, VD1.I/O3, X4.D-
- new net DP3: U$13.DP3, VD2.I/O1, X3.D-
- new net DP4: U$13.DP4, VD2.I/O3, X2.D-
- new net DPU: DATA_USB.D+, U$13.DPU, VD3.I/O4
- new net N$64: D3.A, PAD1.P
- new net N$65: C21.2, D1.C, L1.2, U$12.SW
- new net N$66: C21.1, U$12.BS
- new net N$67: C22.2, R2.1
- new net N$68: C22.1, U$12.COMP
- new net N$69: R3.1, R9.2, U$12.FB
- new net N$70: C31.2, U$13.VD33, U$13.VD33_O
- new net N$71: C30.2, U$13.VD18, U$13.VD18_O
- new net N$72: R10.2, U$13.REXT
- new net N$73: R13.2, U$13.XRSTJ
- new net N$74: R11.2, U$13.BUSJ
- new net N$75: C33.1, Q1.2, U$13.XOUT
- new net N$76: C34.1, Q1.1, U$13.XIN
- new net N$77: LED6.C, R19.1
- new net N$78: LED4.C, LED5.A, R15.1
- new net N$79: LED2.A, LED3.C, R14.1
- new net N$80: LED2.C, LED3.A, LED4.A, LED5.C, LED6.A, U$13.DRV
- new net N$81: R14.2, U$13.LED2
- new net N$82: R15.2, U$13.LED1
- new net VCC: C26.2, C27.2, C28.2, C29.2, C32.2, D4.C, R11.1, R13.1, R9.1, U$13.OVCJ, U$13.PWRJ, U$13.VDD5, VD1.VBUS, VD2.VBUS, VD3.VBUS, X2.GND, X3.GND, X4.GND, X5.GND
- new net VIN: C25.2, D3.C, U$12.IN
- new net V_UP: DATA_USB.VBUS, U$13.VBUSM
- net GND: now also C23.1, C24.1, C25.1, C26.1, C27.1, C28.1, C29.1, C30.1, C31.1, C32.1, C33.2, C34.2, D1.A, DATA_USB.GND, J1.GND@1, J1.GND@10, J1.GND@2, J1.GND@3, J1.GND@4, J1.GND@5, J1.GND@7, J1.GND@8, J1.GND@9, PAD2.P, R10.1, R19.2, R3.2, U$12.GND, U$13.VSS, VD1.GND, VD2.GND, VD3.GND, X2.VBUS, X3.VBUS, X4.VBUS, X5.VBUS; no longer J1._GND@1, J1._GND@10, J1._GND@2, J1._GND@3, J1._GND@4, J1._GND@5, J1._GND@7, J1._GND@8, J1._GND@9
Other:
- note added: "Close left = input is already 5V Close right = input is 7 - 28V"
- note added: "Downstream"
- note added: "LEDs"
- note added: "Port 1"
- note added: "Port 2"
- note added: "Port 3"
- note added: "Port 4"
- note added: "Power"
- note added: "Power supply 1"
- note added: "USB Hub"
- note added: "Upstream"
